Commit message: Add comment, Change the base link hight

File: cart_pole_v2.urdf (robot description, URDF)
Before this commit: robot cart_pole, 6 links, 5 joints
Links:
- link base_left_wall: geometry collision box size=0.2 0.2 1.0; visual box size=0.2 0.2 1.0
- link base_right_wall: geometry collision box size=0.2 0.2 1.0; visual box size=0.2 0.2 1.0
Joints:
- joint base_to_left_wall: origin xyz=-2.4 0 -0.45 -> xyz=-2.4 0 -0.5
- joint base_to_right_wall: origin xyz=2.4 0 -0.45 -> xyz=2.4 0 -0.5

Commit message: Change the mass of pole

File: cart_pole_v2.urdf (robot description, URDF)
Before this commit: robot cart_pole, 6 links, 5 joints
Links:
- link pole: mass 1.0 -> 3.0
